Commit message: kinematics model

File: milling_robot_description/urdf/milling_robot.urdf (robot description, URDF)
Before this commit: robot milling_robot, 5 links, 4 joints
Joints:
- joint D4: limit lower=-0.008 upper=0.02 effort=1000.0 velocity=0.5 -> lower=0.0 upper=0.03 effort=1000.0 velocity=0.5

Commit message: new robot urdf with correct init pose

File: milling_robot_description/urdf/milling_robot.urdf (robot description, URDF)
Before this commit: robot milling_robot, 5 links, 4 joints
Links:
- added link Gripper1, mass 0.0001435229790341507; collision mesh filename=package://milling_robot_description/meshes/Gripper1.stl scale=0.001 0.001 0.001; visual mesh filename=package://milling_robot_description/meshes/Gripper1.stl scale=0.001 0.001 0.001
- added link Gripper2, mass 0.00014352299037443815; collision mesh filename=package://milling_robot_description/meshes/Gripper2.stl scale=0.001 0.001 0.001; visual mesh filename=package://milling_robot_description/meshes/Gripper2.stl scale=0.001 0.001 0.001
- link link2: mass 0.021696703597929294 -> 0.02169670359792929
- link link4: mass 0.003623226210979948 -> 0.003336180247396665
Joints:
- added joint G1: type prismatic, parent link4, child Gripper1, origin xyz=-0.006 -0.002 0.001 rpy=0 0 0, axis 1.0 -0.0 -0.0, limit lower=0.0 upper=0.006 effort=1000.0 velocity=0.5
- added joint G2: type prismatic, parent link4, child Gripper2, origin xyz=0.006 -0.002 0.001 rpy=0 0 0, axis -1.0 -0.0 -0.0, limit lower=0.0 upper=0.006 effort=1000.0 velocity=0.5
- joint D4: axis 0.0 -1.0 0.0 -> 0.0 -0.0 1.0; origin xyz=0.0 0.0 0.0 rpy=0 0 0 -> xyz=0.0 0.0 0.005 rpy=0 0 0
- joint Q3: axis 0.0 -1.0 0.0 -> 0.0 -0.0 1.0; origin xyz=-0.003 -0.037 0.0 rpy=0 0 0 -> xyz=-0.003 0.0 0.037 rpy=0 0 0
